File: hw/esp32.sch (KiCad schematic (older format))
At the start: 0 parts

Commit message: add esp32 and IMU components to schematics
Parts:
- added U?: ESP32, QFN48-0.4MM, symbol ESP32-WROOM-32D:ESP32
Changed lines of the file:
@@
 Comment4 "Component Prefix: ESP"
 $EndDescr
+$Comp
+L ESP32-WROOM-32D:ESP32 U?
+U 1 1 6099F0F4
+P 5100 4150
+F 0 "U?" H 5100 5917 50  0000 C CNN
+F 1 "ESP32" H 5100 5826 50  0000 C CNN
+F 2 "QFN48-0.4MM" H 5100 4150 50  0001 L BNN
+F 3 "" H 5100 4150 50  0001 L BNN
+F 4 "IC-13338" H 5100 4150 50  0001 L BNN "PROD_ID"
+	1    5100 4150
+	1    0    0    -1
+$EndComp
 $EndSCHEMATC

Commit message: Modified ESP32 and IMU symbol properties. Generated netlist and tables as example
Parts:
- removed U?: ESP32, QFN48-0.4MM, symbol ESP32-WROOM-32D:ESP32
- added U1: ESP32, footprints:ESP32-WROOM-32D, symbol ESP32-WROOM-32D:ESP32
Changed lines of the file:
@@
 $EndDescr
 $Comp
-L ESP32-WROOM-32D:ESP32 U?
-U 1 1 6099F0F4
-P 5100 4150
-F 0 "U?" H 5100 5917 50  0000 C CNN
-F 1 "ESP32" H 5100 5826 50  0000 C CNN
-F 2 "QFN48-0.4MM" H 5100 4150 50  0001 L BNN
-F 3 "" H 5100 4150 50  0001 L BNN
-F 4 "IC-13338" H 5100 4150 50  0001 L BNN "PROD_ID"
-	1    5100 4150
+L ESP32-WROOM-32D:ESP32 U1
+U 1 1 609A1D57
+P 5650 3900
+F 0 "U1" H 5650 6121 50  0000 C CNN
+F 1 "ESP32" H 5650 6030 50  0000 C CNN
+F 2 "footprints:ESP32-WROOM-32D" H 5650 3900 50  0001 L BNN
+F 3 "https://www.espressif.com/sites/default/files/documentation/esp32-wroom-32d_esp32-wroom-32u_datasheet_en.pdf" H 5650 5939 50  0000 C CNN
+F 4 "IC-13338" H 5650 3900 50  0001 L BNN "PROD_ID"
+F 5 "1965-ESP32-WROOM-32U(4MB)TR-ND" H 5650 5848 50  0000 C CNN "Vendor Part Number"
+F 6 "Espressif Systems" H 5650 5757 50  0000 C CNN "Manufacturer"
+F 7 "ESP32-WROOM-32U (4MB)" H 5650 5666 50  0000 C CNN "Manufacturer Product Number"
+F 8 "Digikey Canada" H 5650 5575 50  0000 C CNN "Vendor"
+	1    5650 3900
 	1    0    0    -1
 $EndComp

Commit message: Updated schematics and footprints to use default shared libraries. Updated general schematic
Parts:
- removed U1: ESP32, footprints:ESP32-WROOM-32D, symbol ESP32-WROOM-32D:ESP32
- added U_ESP_1: ESP32-WROOM-32D, RF_Module:ESP32-WROOM-32, symbol RF_Module:ESP32-WROOM-32D
Changed lines of the file:
@@
 $EndDescr
 $Comp
-L ESP32-WROOM-32D:ESP32 U1
-U 1 1 609A1D57
-P 5650 3900
-F 0 "U1" H 5650 6121 50  0000 C CNN
-F 1 "ESP32" H 5650 6030 50  0000 C CNN
-F 2 "footprints:ESP32-WROOM-32D" H 5650 3900 50  0001 L BNN
-F 3 "https://www.espressif.com/sites/default/files/documentation/esp32-wroom-32d_esp32-wroom-32u_datasheet_en.pdf" H 5650 5939 50  0000 C CNN
-F 4 "IC-13338" H 5650 3900 50  0001 L BNN "PROD_ID"
-F 5 "1965-ESP32-WROOM-32U(4MB)TR-ND" H 5650 5848 50  0000 C CNN "Vendor Part Number"
-F 6 "Espressif Systems" H 5650 5757 50  0000 C CNN "Manufacturer"
-F 7 "ESP32-WROOM-32U (4MB)" H 5650 5666 50  0000 C CNN "Manufacturer Product Number"
-F 8 "Digikey Canada" H 5650 5575 50  0000 C CNN "Vendor"
-	1    5650 3900
+L RF_Module:ESP32-WROOM-32D U_ESP_1
+U 1 1 609A3F69
+P 5050 3400
+F 0 "U_ESP_1" H 5050 4981 50  0000 C CNN
+F 1 "ESP32-WROOM-32D" H 5050 4890 50  0000 C CNN
+F 2 "RF_Module:ESP32-WROOM-32" H 5050 1900 50  0001 C CNN
+F 3 "https://www.espressif.com/sites/default/files/documentation/esp32-wroom-32d_esp32-wroom-32u_datasheet_en.pdf" H 4750 3450 50  0001 C CNN
+F 4 "	‎Espressif Systems‎" H 5050 3400 50  0001 C CNN "Manufacturer"
+F 5 "ESP32-WROOM-32D (16MB)" H 5050 3400 50  0001 C CNN "Manufacturer Product Number"
+F 6 "Digikey Canada" H 5050 3400 50  0001 C CNN "Vendor"
+F 7 "1904-1025-1-ND" H 5050 3400 50  0001 C CNN "Vendor Product Number"
+	1    5050 3400
 	1    0    0    -1
 $EndComp

Commit message: minor changes
Connections:
- net labels added: GND, IMU_INT1, IMU_INT2, IMU_SCL, IMU_SDA, IMU_SDO
- wire segments 0 -> 6
Changed lines of the file:
@@
 	1    0    0    -1
 $EndComp
+$Comp
+L power:GND #PWR?
+U 1 1 60AB04B1
+P 5050 5050
+F 0 "#PWR?" H 5050 4800 50  0001 C CNN
+F 1 "GND" H 5055 4877 50  0000 C CNN
+F 2 "" H 5050 5050 50  0001 C CNN
+F 3 "" H 5050 5050 50  0001 C CNN
+	1    5050 5050
+	1    0    0    -1
+$EndComp
+Wire Wire Line
+	5050 4800 5050 5050
+Text HLabel 6350 3500 2    50   Input ~ 0
+IMU_SDO
+Text HLabel 6350 3400 2    50   Input ~ 0
+IMU_INT1
+Text HLabel 6350 3300 2    50   Input ~ 0
+IMU_INT2
+Text HLabel 6350 3700 2    50   Output ~ 0
+IMU_SCL
+Text HLabel 6350 3600 2    50   Input ~ 0
+IMU_SDA
+Wire Wire Line
+	5650 3300 6350 3300
+Wire Wire Line
+	5650 3400 6350 3400
+Wire Wire Line
+	5650 3500 6350 3500
+Wire Wire Line
+	5650 3600 6350 3600
+Wire Wire Line
+	5650 3700 6350 3700
 $EndSCHEMATC
