File: hw/esp32.sch (KiCad schematic (older format))
At the start: 1 part

Commit message: Routing headers to ESP32/ Added peripherals
Adopted to peripheral of https://www.espressif.com/sites/default/files/documentation/esp32-wroom-32d_esp32-wroom-32u_datasheet_en.pdf
Parts:
- removed U_ESP_1: ESP32-WROOM-32D, RF_Module:ESP32-WROOM-32, symbol RF_Module:ESP32-WROOM-32D
- added C_ESP_1, C_ESP_2: 0.1uF, symbol Device:C
- added C_ESP_1: 10uF, symbol Device:C
- added PIN_1_ESP: Conn_01x20_Female, symbol Connector:Conn_01x20_Female
- added PIN_2_ESP: Conn_01x15_Female, symbol Connector:Conn_01x15_Female
- added PIN_2_ESP: Conn_01x14_Female, symbol Connector:Conn_01x14_Female
- added R_ESP_1: 10k, symbol Device:R_Small
- added R_ESP_2: 1k, symbol Device:R_Small
- added SW?: PTS647SK38SMTR2LFS, PTS647SK38SMTR2LFS_CNK, symbol PTS647SK38SMTR2LFS:PTS647SK38SMTR2LFS
Connections:
- net labels added: +3.3V, 3V3, EN, GND, IO0, IO12, IO13, IO14, IO15, IO16, IO17, IO18, IO19, IO2, IO21, IO22, IO23, IO25, IO26, IO27, IO32, IO33, IO34, IO35, IO4, IO5, RXD0, SCK, SCS, SDI, SDO, SENSOR_VN, SENSOR_VP, SHD, SWP, TXD0
- wire segments 0 -> 108
- no-connect marks 0 -> 1
Other:
- note added: "Maybe attach it to the base (metal) and have a metal strip rubbing the ground."
- note added: "This would discharge and ground the device. Would also combat the static that is generated by the tires"
- note added: "U2 would go here (substituted by header pins)"
- note added: "Would you like to have a pinout for ground to lead to a larger grounding device?"

Commit message: Combining the ESP and IMU Modules
Parts:
- removed PIN_2_ESP: Conn_01x15_Female, symbol Connector:Conn_01x15_Female
- SW?: symbol PTS647SK38SMTR2LFS:PTS647SK38SMTR2LFS -> rover_controller-rescue:PTS647SK38SMTR2LFS-PTS647SK38SMTR2LFS
Connections:
- net labels added: IMU_SCL, IMU_SD0_SA0, IMU_SDA
- wire segments 108 -> 96
Other:
- note removed: "Maybe attach it to the base (metal) and have a metal strip rubbing the ground."
- note removed: "This would discharge and ground the device. Would also combat the static that is generated by the tires"
- note removed: "Would you like to have a pinout for ground to lead to a larger grounding device?"

Commit message: Finalized the Pins and Connectors
Included the SCL, SDA, SD0_SA0 and interrupts and header pins to jump the connections
Connections:
- net labels added: IMU_INT1, IMU_INT2
- wire segments 96 -> 98
Changed lines of the file:
@@
 	3850 4350 3400 4350
-Wire Wire Line
-	3850 4450 3400 4450
 Wire Wire Line
 	3850 4550 3400 4550
@@
 Text Label 3400 4350 0    50   ~ 0
 IO32
-Text Label 3400 4450 0    50   ~ 0
-IO25
 Text Label 3400 4550 0    50   ~ 0
 IO26
@@
 Text HLabel 7500 5650 2    50   Output ~ 0
 IMU_SCL
+Wire Wire Line
+	7150 5750 7500 5750
+Wire Wire Line
+	7150 5850 7500 5850
+Text Label 7150 5750 2    50   ~ 0
+IO26
+Text Label 3400 4450 0    50   ~ 0
+IO25
+Wire Wire Line
+	3850 4450 3400 4450
+Text Label 7150 5850 2    50   ~ 0
+IO25
+Text HLabel 7500 5750 2    50   Output ~ 0
+IMU_INT2
+Text HLabel 7500 5850 2    50   Output ~ 0
+IMU_INT1
 $EndSCHEMATC
