File: hw/rover_controller.sch (KiCad schematic (older format))
At the start: 0 parts

Commit message: minor changes
Changed lines of the file:
@@
 $EndDescr
 $Sheet
-S 4850 2500 1050 1150
+S 4700 2200 1150 1850
 U 6099F001
 F0 "ESP32" 50
 F1 "esp32.sch" 50
+F2 "INT1_IMU" O R 5850 3600 50
+F3 "INT2_IMU" O R 5850 3350 50
+F4 "SCL_IMU" O R 5850 3100 50
+F5 "SDA_IMU" I R 5850 2850 50
+F6 "SDO_IMU_IN" I R 5850 2600 50
 $EndSheet
 $Sheet
-S 6700 2600 950  900
+S 7050 2500 1150 1200
 U 6099FD27
 F0 "IMU" 50
 F1 "imu.sch" 50
+F2 "IMU_SDA" O L 7050 2850 50
+F3 "IMU_INT1" I L 7050 3600 50
+F4 "IMU_SDO_SA0" O L 7050 2600 50
+F5 "IMU_SCL" I L 7050 3100 50
+F6 "IMU_INT2" I L 7050 3350 50
 $EndSheet
+Wire Wire Line
+	5850 2600 7050 2600
+Wire Wire Line
+	5850 2850 7050 2850
+Wire Wire Line
+	5850 3100 7050 3100
+Wire Wire Line
+	5850 3350 7050 3350
+Wire Wire Line
+	5850 3600 7050 3600
 $EndSCHEMATC
