File: hw/rover_controller.sch (KiCad schematic (older format))
At the start: 0 parts

Commit message: Combining the ESP and IMU Modules
Parts:
- added J_RC_1: Conn_01x05_Female, symbol Connector:Conn_01x05_Female
Connections:
- wire segments 5 -> 10
Changed lines of the file:
@@
 $EndDescr
 $Sheet
-S 4700 2200 1150 1850
+S 5350 2100 1150 1850
 U 6099F001
 F0 "ESP32" 50
 F1 "esp32.sch" 50
-F2 "INT1_IMU" O R 5850 3600 50
-F3 "INT2_IMU" O R 5850 3350 50
-F4 "SCL_IMU" O R 5850 3100 50
-F5 "SDA_IMU" I R 5850 2850 50
-F6 "SDO_IMU_IN" I R 5850 2600 50
+F2 "IMU_SD0_SA0" O R 6500 3000 50
+F3 "IMU_SDA" B R 6500 2750 50
+F4 "IMU_SCL" O R 6500 2500 50
 $EndSheet
+Wire Wire Line
+	6500 2500 7700 2500
+Wire Wire Line
+	6500 2750 7700 2750
+Wire Wire Line
+	6500 3000 7700 3000
+Wire Wire Line
+	6500 3250 7700 3250
+Wire Wire Line
+	6500 3500 7700 3500
 $Sheet
-S 7050 2500 1150 1200
+S 7700 2400 1150 1200
 U 6099FD27
 F0 "IMU" 50
 F1 "imu.sch" 50
-F2 "IMU_SDA" O L 7050 2850 50
-F3 "IMU_INT1" I L 7050 3600 50
-F4 "IMU_SDO_SA0" O L 7050 2600 50
-F5 "IMU_SCL" I L 7050 3100 50
-F6 "IMU_INT2" I L 7050 3350 50
+F2 "IMU_INT1" I L 7700 3500 50
+F3 "IMU_INT2" I L 7700 3250 50
+F4 "IMU_SCL" I L 7700 2500 50
+F5 "IMU_SDA" B L 7700 2750 50
+F6 "IMU_SDO_SA0" I L 7700 3000 50
 $EndSheet
+$Comp
+L Connector:Conn_01x05_Female J_RC_1
+U 1 1 60DCA10D
+P 3850 3000
+F 0 "J_RC_1" H 3742 3385 50  0000 C CNN
+F 1 "Conn_01x05_Female" H 3742 3294 50  0000 C CNN
+F 2 "" H 3850 3000 50  0001 C CNN
+F 3 "~" H 3850 3000 50  0001 C CNN
+	1    3850 3000
+	-1   0    0    -1
+$EndComp
 Wire Wire Line
-	5850 2600 7050 2600
+	4050 2800 4350 2800
 Wire Wire Line
-	5850 2850 7050 2850
+	4050 2900 4350 2900
 Wire Wire Line
-	5850 3100 7050 3100
+	4050 3000 4350 3000
 Wire Wire Line
-	5850 3350 7050 3350
+	4050 3100 4350 3100
 Wire Wire Line
-	5850 3600 7050 3600
+	4050 3200 4350 3200
 $EndSCHEMATC

Commit message: Finalized the Pins and Connectors
Included the SCL, SDA, SD0_SA0 and interrupts and header pins to jump the connections
Parts:
- removed J_RC_1: Conn_01x05_Female, symbol Connector:Conn_01x05_Female
- added J_RC_INT1, J_RC_INT2, J_RC_SCL, J_RC_SD0_SA0, J_RC_SDA: Conn_01x02_Female, symbol Connector:Conn_01x02_Female
Connections:
- net labels added: INT1_ESP_O, INT1_IMU_I, INT2_ESP_O, INT2_IMU_I, SCL_ESP_O, SCL_IMU_I, SD0_SA0_ESP_O, SD0_SA0_IMU_I, SDA_ESP_O, SDA_IMU_I
- wire segments 10 -> 20
Changed lines of the file:
@@
 $EndDescr
 $Sheet
-S 5350 2100 1150 1850
+S 4600 2100 1150 1850
 U 6099F001
 F0 "ESP32" 50
 F1 "esp32.sch" 50
-F2 "IMU_SD0_SA0" O R 6500 3000 50
-F3 "IMU_SDA" B R 6500 2750 50
-F4 "IMU_SCL" O R 6500 2500 50
+F2 "IMU_SD0_SA0" O R 5750 3000 50
+F3 "IMU_SDA" B R 5750 2750 50
+F4 "IMU_SCL" O R 5750 2500 50
+F5 "IMU_INT2" O R 5750 3250 50
+F6 "IMU_INT1" O R 5750 3500 50
 $EndSheet
-Wire Wire Line
-	6500 2500 7700 2500
-Wire Wire Line
-	6500 2750 7700 2750
-Wire Wire Line
-	6500 3000 7700 3000
-Wire Wire Line
-	6500 3250 7700 3250
-Wire Wire Line
-	6500 3500 7700 3500
 $Sheet
 S 7700 2400 1150 1200
@@
 F6 "IMU_SDO_SA0" I L 7700 3000 50
 $EndSheet
+Wire Wire Line
+	5750 2500 6050 2500
+Wire Wire Line
+	5750 2750 6050 2750
+Wire Wire Line
+	5750 3000 6050 3000
+Wire Wire Line
+	5750 3250 6050 3250
+Wire Wire Line
+	5750 3500 6050 3500
+Wire Wire Line
+	7400 2500 7700 2500
+Wire Wire Line
+	7400 2750 7700 2750
+Wire Wire Line
+	7400 3000 7700 3000
+Wire Wire Line
+	7400 3250 7700 3250
+Wire Wire Line
+	7400 3500 7700 3500
+Text Label 6050 2500 0    50   ~ 0
+SCL_ESP_O
+Text Label 6050 3250 0    50   ~ 0
+INT2_ESP_O
+Text Label 6050 3500 0    50   ~ 0
+INT1_ESP_O
+Text Label 6050 2750 0    50   ~ 0
+SDA_ESP_O
+Text Label 6050 3000 0    50   ~ 0
+SD0_SA0_ESP_O
+Text Label 7400 2500 2    50   ~ 0
+SCL_IMU_I
+Text Label 7400 2750 2    50   ~ 0
+SDA_IMU_I
+Text Label 7400 3000 2    50   ~ 0
+SD0_SA0_IMU_I
+Text Label 7400 3250 2    50   ~ 0
+INT2_IMU_I
+Text Label 7400 3500 2    50   ~ 0
+INT1_IMU_I
 $Comp
-L Connector:Conn_01x05_Female J_RC_1
-U 1 1 60DCA10D
-P 3850 3000
-F 0 "J_RC_1" H 3742 3385 50  0000 C CNN
-F 1 "Conn_01x05_Female" H 3742 3294 50  0000 C CNN
-F 2 "" H 3850 3000 50  0001 C CNN
-F 3 "~" H 3850 3000 50  0001 C CNN
-	1    3850 3000
-	-1   0    0    -1
+L Connector:Conn_01x02_Female J_RC_SDA
+U 1 1 60DE5F30
+P 2500 2500
+F 0 "J_RC_SDA" H 2528 2476 50  0000 L CNN
+F 1 "Conn_01x02_Female" H 2528 2385 50  0000 L CNN
+F 2 "" H 2500 2500 50  0001 C CNN
+F 3 "~" H 2500 2500 50  0001 C CNN
+	1    2500 2500
+	1    0    0    -1
+$EndComp
+$Comp
+L Connector:Conn_01x02_Female J_RC_SD0_SA0
+U 1 1 60DE63B8
+P 2500 3150
+F 0 "J_RC_SD0_SA0" H 2528 3126 50  0000 L CNN
+F 1 "Conn_01x02_Female" H 2528 3035 50  0000 L CNN
+F 2 "" H 2500 3150 50  0001 C CNN
+F 3 "~" H 2500 3150 50  0001 C CNN
+	1    2500 3150
+	1    0    0    -1
+$EndComp
+$Comp
+L Connector:Conn_01x02_Female J_RC_INT2
+U 1 1 60DE6BC0
+P 2500 3850
+F 0 "J_RC_INT2" H 2528 3826 50  0000 L CNN
+F 1 "Conn_01x02_Female" H 2528 3735 50  0000 L CNN
+F 2 "" H 2500 3850 50  0001 C CNN
+F 3 "~" H 2500 3850 50  0001 C CNN
+	1    2500 3850
+	1    0    0    -1
+$EndComp
+$Comp
+L Connector:Conn_01x02_Female J_RC_INT1
+U 1 1 60DE6FA4
+P 2500 4500
+F 0 "J_RC_INT1" H 2528 4476 50  0000 L CNN
+F 1 "Conn_01x02_Female" H 2528 4385 50  0000 L CNN
+F 2 "" H 2500 4500 50  0001 C CNN
+F 3 "~" H 2500 4500 50  0001 C CNN
+	1    2500 4500
+	1    0    0    -1
+$EndComp
+$Comp
+L Connector:Conn_01x02_Female J_RC_SCL
+U 1 1 60DE4977
+P 2500 1800
+F 0 "J_RC_SCL" H 2528 1776 50  0000 L CNN
+F 1 "Conn_01x02_Female" H 2528 1685 50  0000 L CNN
+F 2 "" H 2500 1800 50  0001 C CNN
+F 3 "~" H 2500 1800 50  0001 C CNN
+	1    2500 1800
+	1    0    0    -1
 $EndComp
 Wire Wire Line
-	4050 2800 4350 2800
+	2300 1800 2000 1800
+Text Label 2000 1800 2    50   ~ 0
+SCL_ESP_O
 Wire Wire Line
-	4050 2900 4350 2900
+	2000 1900 2300 1900
+Text Label 2000 1900 2    50   ~ 0
+SCL_IMU_I
 Wire Wire Line
-	4050 3000 4350 3000
+	2000 2600 2300 2600
+Text Label 2000 2600 2    50   ~ 0
+SDA_IMU_I
 Wire Wire Line
-	4050 3100 4350 3100
+	2000 3250 2300 3250
+Text Label 2000 3250 2    50   ~ 0
+SD0_SA0_IMU_I
 Wire Wire Line
-	4050 3200 4350 3200
+	2000 3950 2300 3950
+Text Label 2000 3950 2    50   ~ 0
+INT2_IMU_I
+Wire Wire Line
+	2000 4600 2300 4600
+Text Label 2000 4600 2    50   ~ 0
+INT1_IMU_I
+Wire Wire Line
+	2300 2500 2000 2500
+Text Label 2000 2500 2    50   ~ 0
+SDA_ESP_O
+Wire Wire Line
+	2300 3150 2000 3150
+Text Label 2000 3150 2    50   ~ 0
+SD0_SA0_ESP_O
+Wire Wire Line
+	2300 3850 2000 3850
+Text Label 2000 3850 2    50   ~ 0
+INT2_ESP_O
+Wire Wire Line
+	2300 4500 2000 4500
+Text Label 2000 4500 2    50   ~ 0
+INT1_ESP_O
 $EndSCHEMATC
